File: Toad'sTempest.kicad_sch (KiCad schematic)
At the start: 109 parts, among them J1 USB_C_Receptacle_USB2.0, SW1 SW_Push, SW10 SW_Push, SW11 SW_Push, SW12 SW_Push, SW13 SW_Push, SW14 SW_Push, SW15 SW_Push, SW16 SW_Push, SW17 SW_Push, SW18 SW_Push, SW19 SW_Push, SW2 SW_Push, SW20 SW_Push, SW21 SW_Push, SW22 SW_Push, SW23 SW_Push, SW24 SW_Push, SW25 SW_Push, SW26 SW_Push, SW27 SW_Push, SW28 SW_Push, SW29 SW_Push, SW3 SW_Push, SW30 SW_Push, SW31 SW_Push, SW32 SW_Push, SW33 SW_Push, SW34 SW_Push, SW35 SW_Push, SW36 SW_Push, SW37 SW_Push, SW38 SW_Push, SW39 SW_Push, SW4 SW_Push, SW40 SW_Push, SW41 SW_Push, SW42 SW_Push, SW43 BOOT, SW44 RESET, SW5 SW_Push, SW6 SW_Push, SW7 SW_Push, SW8 SW_Push, SW9 SW_Push, U1 USBLC6-2SC6, U2 CH552T

Commit message: upd readme
Other:
- company: (none) -> T1K1N$0N
- title: (none) -> "Toad'sTempest" mechanical keyboard
Changed lines of the file:
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@@
 	(generator_version "8.0")
 	(paper "A3")
+	(title_block
+		(title "\"Toad'sTempest\" mechanical keyboard")
+		(company "T1K1N$0N")
+		(comment 1 "https://github.com/tikinson/ToadsTempest")
+	)
 	(junction
 		(at 90.17 120.65)
